File: PCB/Nifty Numpad.kicad_sch (KiCad schematic)
At the start: 43 parts, among them J101 SWD, J102 USB-C, J103 UART, SW101 PTS636 SL43 SMTR LFS, SW102 PTS636 SL43 SMTR LFS, U101 MIC5366-3.3YC5, U102 CM1213A−02Sx, U103 SN74LVC1T45DCK, U104 RP2040, U105 W25Q40CLSNIG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

Commit message: Fixed LED rotation, beefed up standoffs, added docs
Parts:
- H101, H102, H103, H104, H105: footprint irex_MountingHole:MountingHole_4.6mm_ReducedCourtyard -> irex_MountingHole:MountingHole_6.0mm_ReducedCourtyard
Changed lines of the file:
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@@
     (title "Nifty Numpad")
     (date "2023-06-10")
-    (rev "0")
+    (rev "${REV}")
     (comment 1 "Isaac Rex")
   )
@@
       (effects (font (size 1.27 1.27)) (justify left))
     )
-    (property "Footprint" "irex_MountingHole:MountingHole_4.6mm_ReducedCourtyard" (at 146.05 27.94 0)
+    (property "Footprint" "irex_MountingHole:MountingHole_6.0mm_ReducedCourtyard" (at 146.05 27.94 0)
       (effects (font (size 1.27 1.27)) hide)
     )
@@
       (effects (font (size 1.27 1.27)) (justify left))
     )
-    (property "Footprint" "irex_MountingHole:MountingHole_4.6mm_ReducedCourtyard" (at 161.29 19.05 0)
+    (property "Footprint" "irex_MountingHole:MountingHole_6.0mm_ReducedCourtyard" (at 161.29 19.05 0)
       (effects (font (size 1.27 1.27)) hide)
     )
@@
       (effects (font (size 1.27 1.27)) (justify left))
     )
-    (property "Footprint" "irex_MountingHole:MountingHole_4.6mm_ReducedCourtyard" (at 130.81 19.05 0)
+    (property "Footprint" "irex_MountingHole:MountingHole_6.0mm_ReducedCourtyard" (at 130.81 19.05 0)
       (effects (font (size 1.27 1.27)) hide)
     )
@@
       (effects (font (size 1.27 1.27)) (justify left))
     )
-    (property "Footprint" "irex_MountingHole:MountingHole_4.6mm_ReducedCourtyard" (at 130.81 27.94 0)
+    (property "Footprint" "irex_MountingHole:MountingHole_6.0mm_ReducedCourtyard" (at 130.81 27.94 0)
       (effects (font (size 1.27 1.27)) hide)
     )
@@
       (effects (font (size 1.27 1.27)) (justify left))
     )
-    (property "Footprint" "irex_MountingHole:MountingHole_4.6mm_ReducedCourtyard" (at 146.05 19.05 0)
+    (property "Footprint" "irex_MountingHole:MountingHole_6.0mm_ReducedCourtyard" (at 146.05 19.05 0)
       (effects (font (size 1.27 1.27)) hide)
     )
